Commit message: 1

File: description/robot_core.xacro (robot description, xacro)
@@ -1,46 +1,23 @@
 <?xml version="1.0"?>
-<robot xmlns:xacro="http://www.ros.org/wiki/xacro" >
-    <!--<xacro:include filename="inertial_macros.xacro"/>-->
-    <xacro:property name="chassis_length" value="0.335"/>
-    <xacro:property name="chassis_width" value="0.265"/>
-    <xacro:property name="chassis_height" value="0.138"/>
+<robot xmlns:xacro="http://www.ros.org/wiki/xacro">
+    <xacro:property name="chassis_length" value="0.360"/>
+    <xacro:property name="chassis_width" value="0.200"/>
+    <xacro:property name="chassis_height" value="0.100"/>
     <xacro:property name="chassis_mass" value="1.0"/>
-    <xacro:property name="wheel_radius" value="0.033"/>
-    <xacro:property name="wheel_thickness" value="0.026"/>
+    <xacro:property name="wheel_radius" value="0.0675"/>
+    <xacro:property name="wheel_thickness" value="0.043"/>
     <xacro:property name="wheel_mass" value="0.05"/>
     <xacro:property name="wheel_offset_x" value="0.226"/>
     <xacro:property name="wheel_offset_y" value="0.1485"/>
     <xacro:property name="wheel_offset_z" value="0.01"/>
-    <xacro:property name="caster_wheel_radius" value="0.01"/>
-    <xacro:property name="caster_wheel_mass" value="0.01"/>
-    <xacro:property name="caster_wheel_offset_x" value="0.075"/>
-    <xacro:property name="caster_wheel_offset_z" value="${wheel_offset_z - wheel_radius + caster_wheel_radius}"/>
-    <material name="white">
-        <color rgba="1 1 1 1" />
+    <material name="black">
+        <color rgba="0 0 0 1"/>
     </material>
     <material name="orange">
         <color rgba="1 0.3 0.1 1"/>
     </material>
-    <material name="blue">
-        <color rgba="0.2 0.2 1 1"/>
-    </material>
-    <material name="black">
-        <color rgba="0 0 0 1"/>
-    </material>
-    <material name="red">
-        <color rgba="1 0 0 1"/>
-    </material>
-    <!-- BASE LINK -->
-    <link name="base_link">
-    </link>
-    <!-- BASE_FOOTPRINT LINK -->
-    <joint name="base_footprint_joint" type="fixed">
-        <parent link="base_link"/>
-        <child link="base_footprint"/>
-        <origin xyz="0 0 0" rpy="0 0 0"/>
-    </joint>
-    <link name="base_footprint">
-    </link>
-    <!-- CHASSIS LINK -->
+    <!-- Base Link -->
+    <link name="base_link"/>
+    <!-- Chassis -->
     <joint name="chassis_joint" type="fixed">
         <parent link="base_link"/>
@@ -62,96 +39,30 @@
             </geometry>
         </collision>
-        <xacro:inertial_box mass="0.5" x="${chassis_length}" y="${chassis_width}" z="${chassis_height}">
-            <origin xyz="${chassis_length/2} 0 ${chassis_height/2}" rpy="0 0 0"/>
-        </xacro:inertial_box>
     </link>
-<!--
-    <gazebo reference="chassis">
-        <material>Gazebo/Orange</material>
-    </gazebo>
--->
-    <!-- LEFT WHEEL LINK -->
-    <joint name="left_wheel_joint" type="continuous">
-        <parent link="base_link"/>
-        <child link="left_wheel"/>
-        <origin xyz="0 ${wheel_offset_y} 0" rpy="-${pi/2} 0 0" />
-        <axis xyz="0 0 1"/>
-    </joint>
-    <link name="left_wheel">
-        <visual>
-            <geometry>
-                <cylinder radius="${wheel_radius}" length="${wheel_thickness}"/>
-            </geometry>
-            <material name="blue"/>
-        </visual>
-        <collision>
-            <geometry>
-                <sphere radius="${wheel_radius}"/>
-            </geometry>
-        </collision>
-        <xacro:inertial_cylinder mass="${wheel_mass}" length="${wheel_thickness}" radius="${wheel_radius}">
-            <origin xyz="0 0 0" rpy="0 0 0"/>
-        </xacro:inertial_cylinder>
-    </link>
-<!--
-    <gazebo reference="left_wheel">
-        <material>Gazebo/Blue</material>
-    </gazebo>
--->
-    <!-- RIGHT WHEEL LINK -->
-    <joint name="right_wheel_joint" type="continuous">
-        <parent link="base_link"/>
-        <child link="right_wheel"/>
-        <origin xyz="0 ${-wheel_offset_y} 0" rpy="${pi/2} 0 0" />
-        <axis xyz="0 0 -1"/>
-    </joint>
-    <link name="right_wheel">
-        <visual>
-            <geometry>
-                <cylinder radius="${wheel_radius}" length="${wheel_thickness}"/>
-            </geometry>
-            <material name="blue"/>
-        </visual>
-        <collision>
-            <geometry>
-                <sphere radius="${wheel_radius}"/>
-            </geometry>
-        </collision>
-        <xacro:inertial_cylinder mass="${wheel_mass}" length="${wheel_thickness}" radius="${wheel_radius}">
-            <origin xyz="0 0 0" rpy="0 0 0"/>
-        </xacro:inertial_cylinder>
-    </link>
-<!--    <gazebo reference="right_wheel">
-        <material>Gazebo/Blue</material>
-    </gazebo>
--->
-    <!-- CASTER WHEEL LINK -->
-    <joint name="caster_wheel_joint" type="fixed">
-        <parent link="chassis"/>
-        <child link="caster_wheel"/>
-        <origin xyz="${caster_wheel_offset_x} 0 ${caster_wheel_offset_z}"/>
-    </joint>
-    <link name="caster_wheel">
-        <visual>
-            <geometry>
-                <sphere radius="${caster_wheel_radius}"/>
-            </geometry>
-            <material name="white"/>
-        </visual>
-        <collision>
-            <geometry>
-                <sphere radius="${caster_wheel_radius}"/>
-            </geometry>
-        </collision>
-        <xacro:inertial_sphere mass="${caster_wheel_mass}" radius="${caster_wheel_radius}">
-            <origin xyz="0 0 0" rpy="0 0 0"/>
-        </xacro:inertial_sphere>
-    </link>
-<!--
-    <gazebo reference="caster_wheel">
-        <material>Gazebo/White</material>
-        <mu1 value="0.001"/>
-        <mu2 value="0.001"/>
-    </gazebo>
--->
+    <!-- Wheels -->
+    <xacro:macro name="wheel" params="name parent x y z rpy axis">
+        <joint name="${name}_joint" type="continuous">
+            <parent link="${parent}"/>
+            <child link="${name}"/>
+            <origin xyz="${x} ${y} ${z}" rpy="${rpy}"/>
+            <axis xyz="${axis}"/>
+        </joint>
+        <link name="${name}">
+            <visual>
+                <geometry>
+                    <cylinder radius="${wheel_radius}" length="${wheel_thickness}"/>
+                </geometry>
+                <material name="black"/>
+            </visual>
+            <collision>
+                <geometry>
+                    <cylinder radius="${wheel_radius}" length="${wheel_thickness}"/>
+                </geometry>
+            </collision>
+        </link>
+    </xacro:macro>
+    <xacro:wheel name="left_back_wheel" parent="base_link" x="0" y="${wheel_offset_y}" z="0" rpy="-${pi/2} 0 0" axis="0 0 1"/>
+    <xacro:wheel name="left_front_wheel" parent="base_link" x="${wheel_offset_x}" y="${wheel_offset_y}" z="0" rpy="-${pi/2} 0 0" axis="0 0 1"/>
+    <xacro:wheel name="right_back_wheel" parent="base_link" x="0" y="${-wheel_offset_y}" z="0" rpy="${pi/2} 0 0" axis="0 0 -1"/>
+    <xacro:wheel name="right_front_wheel" parent="base_link" x="${wheel_offset_x}" y="${-wheel_offset_y}" z="0" rpy="${pi/2} 0 0" axis="0 0 -1"/>
 </robot>
